Commit message: Auto release sync - 0.8.0
Synchronized at 2026-01-30 19:48:46 UTC with internal commit: c88fc7e2b9e77736fcb0fbe13acbb059196f1796

File: robots/humanoid/vega_1u/vega_1u_f5d6.urdf (robot description, URDF)
Before this commit: robot vega-1, 60 links, 59 joints
Links:
- link L_arm_l1: geometry collision mesh filename=../vega_1/meshes/collision/L_arm_l1.obj; visual mesh filename=../vega_1/meshes/visual/L_arm_l1.glb
- link L_arm_l2: geometry collision mesh filename=../vega_1/meshes/collision/arm_l2.obj; visual mesh filename=../vega_1/meshes/visual/arm_l2.glb
- link L_arm_l3: geometry collision mesh filename=../vega_1/meshes/collision/arm_l3.obj; visual mesh filename=../vega_1/meshes/visual/arm_l3.glb
- link L_arm_l4: geometry collision mesh filename=../vega_1/meshes/collision/arm_l4.obj; visual mesh filename=../vega_1/meshes/visual/arm_l4.glb
- link L_arm_l5: geometry collision mesh filename=../vega_1/meshes/collision/arm_l5.obj; visual mesh filename=../vega_1/meshes/visual/arm_l5.glb
- link L_arm_l6: geometry collision mesh filename=../vega_1/meshes/collision/L_arm_l6.obj; visual mesh filename=../vega_1/meshes/visual/L_arm_l6.glb
- link L_arm_l7: geometry collision mesh filename=../vega_1/meshes/collision/arm_l7.obj; visual mesh filename=../vega_1/meshes/visual/arm_l7.glb
- link L_arm_l8: geometry collision mesh filename=../vega_1/meshes/collision/arm_l8.obj; visual mesh filename=../vega_1/meshes/visual/arm_l8.glb
- link R_arm_l1: geometry collision mesh filename=../vega_1/meshes/collision/R_arm_l1.obj; visual mesh filename=../vega_1/meshes/visual/R_arm_l1.glb
- link R_arm_l2: geometry collision mesh filename=../vega_1/meshes/collision/arm_l2.obj; visual mesh filename=../vega_1/meshes/visual/arm_l2.glb
- link R_arm_l3: geometry collision mesh filename=../vega_1/meshes/collision/arm_l3.obj; visual mesh filename=../vega_1/meshes/visual/arm_l3.glb
- link R_arm_l4: geometry collision mesh filename=../vega_1/meshes/collision/arm_l4.obj; visual mesh filename=../vega_1/meshes/visual/arm_l4.glb
- link R_arm_l5: geometry collision mesh filename=../vega_1/meshes/collision/arm_l5.obj; visual mesh filename=../vega_1/meshes/visual/arm_l5.glb
- link R_arm_l6: geometry collision mesh filename=../vega_1/meshes/collision/R_arm_l6.obj; visual mesh filename=../vega_1/meshes/visual/R_arm_l6.glb
- link R_arm_l7: geometry collision mesh filename=../vega_1/meshes/collision/arm_l7.obj; visual mesh filename=../vega_1/meshes/visual/arm_l7.glb
- link R_arm_l8: geometry collision mesh filename=../vega_1/meshes/collision/arm_l8.obj; visual mesh filename=../vega_1/meshes/visual/arm_l8.glb
- link head_l1: geometry collision mesh filename=../vega_1/meshes/collision/head_l1.obj; visual mesh filename=../vega_1/meshes/visual/head_l1.glb
- link head_l2: geometry collision mesh filename=../vega_1/meshes/collision/head_l2.obj; visual mesh filename=../vega_1/meshes/visual/head_l2.glb
- link head_l3: geometry collision mesh filename=../vega_1/meshes/collision/head_l3.obj; visual mesh filename=../vega_1/meshes/visual/head_l3.glb
- link torso_l3: geometry collision mesh filename=../vega_1/meshes/collision/torso_l3.obj; visual mesh filename=../vega_1/meshes/visual/torso_l3.glb
