Commit message: Auto release sync - 0.8.1
Synchronized at 2026-03-27 00:26:08 UTC with internal commit: db5b9dc937fa2f1801b16b310092b4c2c5aa89ac

File: robots/humanoid/vega_1p/vega_1p.urdf (robot description, URDF)
Before this commit: robot vega_1p, 41 links, 40 joints
Joints:
- joint back_lidar_mount: origin xyz=-0.34 0 0.0985 rpy=1.57079 3.1415 0 -> xyz=-0.34 0 0.0985 rpy=3.14156 0 3.14159
- joint front_lidar_mount: origin xyz=0.306 0 0.287 rpy=3.1415 0 0 -> xyz=0.306 0 0.287 rpy=-0.6981 0 -1.57079

File: robots/humanoid/vega_1p/vega_1p_collision_spheres.collision.urdf (robot description, URDF)
Before this commit: robot vega_1p, 41 links, 40 joints
Joints:
- joint back_lidar_mount: origin xyz=-0.34 0 0.0985 rpy=1.57079 3.1415 0 -> xyz=-0.34 0 0.0985 rpy=3.14156 0 3.14159
- joint front_lidar_mount: origin xyz=0.306 0 0.287 rpy=3.1415 0 0 -> xyz=0.306 0 0.287 rpy=-0.6981 0 -1.57079

File: robots/humanoid/vega_1p/vega_1p_f5d6.urdf (robot description, URDF)
Before this commit: robot vega_1p_f5d6, 75 links, 74 joints
Joints:
- joint back_lidar_mount: origin xyz=-0.34 0 0.0985 rpy=1.57079 3.1415 0 -> xyz=-0.34 0 0.0985 rpy=3.14156 0 3.14159
- joint front_lidar_mount: origin xyz=0.306 0 0.287 rpy=3.1415 0 0 -> xyz=0.306 0 0.287 rpy=-0.6981 0 -1.57079

File: robots/humanoid/vega_1p/vega_1p_f5d6_collision_spheres.collision.urdf (robot description, URDF)
Before this commit: robot vega_1p_f5d6, 75 links, 74 joints
Joints:
- joint back_lidar_mount: origin xyz=-0.34 0 0.0985 rpy=1.57079 3.1415 0 -> xyz=-0.34 0 0.0985 rpy=3.14156 0 3.14159
- joint front_lidar_mount: origin xyz=0.306 0 0.287 rpy=3.1415 0 0 -> xyz=0.306 0 0.287 rpy=-0.6981 0 -1.57079

File: robots/humanoid/vega_1p/vega_1p_gripper.urdf (robot description, URDF)
Before this commit: robot vega_1p_gripper, 47 links, 46 joints
Joints:
- joint back_lidar_mount: origin xyz=-0.34 0 0.0985 rpy=1.57079 3.1415 0 -> xyz=-0.34 0 0.0985 rpy=3.14156 0 3.14159
- joint front_lidar_mount: origin xyz=0.306 0 0.287 rpy=3.1415 0 0 -> xyz=0.306 0 0.287 rpy=-0.6981 0 -1.57079

File: robots/humanoid/vega_1p/vega_1p_gripper_collision_spheres.collision.urdf (robot description, URDF)
Before this commit: robot vega_1p_gripper, 47 links, 46 joints
Joints:
- joint back_lidar_mount: origin xyz=-0.34 0 0.0985 rpy=1.57079 3.1415 0 -> xyz=-0.34 0 0.0985 rpy=3.14156 0 3.14159
- joint front_lidar_mount: origin xyz=0.306 0 0.287 rpy=3.1415 0 0 -> xyz=0.306 0 0.287 rpy=-0.6981 0 -1.57079

File: robots/humanoid/vega_1u/vega_1u.urdf (robot description, URDF)
Before this commit: robot vega_1u, 26 links, 25 joints
Links:
- removed link torso_l3
- added link base_link, mass 18.91029; collision mesh filename=meshes/visual/base_link.glb; visual mesh filename=meshes/visual/base_link.glb
- added link lift_link, mass 4.35777; collision mesh filename=meshes/visual/lift_link.glb; visual mesh filename=meshes/visual/lift_link.glb
- added link torso_flip_link, mass 0.71794; collision mesh filename=meshes/visual/torso_link.glb; visual mesh filename=meshes/visual/torso_link.glb
Joints:
- added joint Lift: type prismatic, parent base_link, child lift_link, origin xyz=0 0 0.01 rpy=0 0 0, axis 0 0 1, limit lower=0 upper=0.4 effort=0 velocity=0.05
- added joint torso_flip: type revolute, parent lift_link, child torso_flip_link, origin xyz=0 -0.06187 0.786 rpy=0 0 0, axis 1 0 0, limit lower=0 upper=1 effort=0 velocity=0.1
- joint arm_center_j0: origin xyz=-0.05908 0 0.44528 rpy=0 0 0 -> xyz=0 0.03852 0.25982 rpy=0 0 -1.57079; parent torso_l3 -> torso_flip_link

File: robots/humanoid/vega_1u/vega_1u_collision_spheres.collision.urdf (robot description, URDF)
Before this commit: robot vega_1u, 26 links, 25 joints
Links:
- removed link torso_l3
- added link base_link, mass 18.91029; visual mesh filename=meshes/visual/base_link.glb
- added link lift_link, mass 4.35777; collision sphere radius=0.09000000357627869; collision sphere radius=0.10999999940395355
- added link torso_flip_link, mass 0.71794; collision sphere radius=0.07999999821186066; collision sphere radius=0.07999999821186066
Joints:
- added joint Lift: type prismatic, parent base_link, child lift_link, origin xyz=0 0 0.01 rpy=0 0 0, axis 0 0 1, limit lower=0 upper=0.4 effort=0 velocity=0.05
- added joint torso_flip: type revolute, parent lift_link, child torso_flip_link, origin xyz=0 -0.06187 0.786 rpy=0 0 0, axis 1 0 0, limit lower=0 upper=1 effort=0 velocity=0.1
- joint arm_center_j0: origin xyz=-0.05908 0 0.44528 rpy=0 0 0 -> xyz=0 0.03852 0.25982 rpy=0 0 -1.57079; parent torso_l3 -> torso_flip_link

File: robots/humanoid/vega_1u/vega_1u_f5d6.urdf (robot description, URDF)
Before this commit: robot vega_1u_f5d6, 60 links, 59 joints
Links:
- removed link torso_l3
- added link base_link, mass 18.91029; collision mesh filename=meshes/visual/base_link.glb; visual mesh filename=meshes/visual/base_link.glb
- added link lift_link, mass 4.35777; collision mesh filename=meshes/visual/lift_link.glb; visual mesh filename=meshes/visual/lift_link.glb
- added link torso_flip_link, mass 0.71794; collision mesh filename=meshes/visual/torso_link.glb; visual mesh filename=meshes/visual/torso_link.glb
Joints:
- added joint Lift: type prismatic, parent base_link, child lift_link, origin xyz=0 0 0.01 rpy=0 0 0, axis 0 0 1, limit lower=0 upper=0.4 effort=0 velocity=0.05
- added joint torso_flip: type revolute, parent lift_link, child torso_flip_link, origin xyz=0 -0.06187 0.786 rpy=0 0 0, axis 1 0 0, limit lower=0 upper=1 effort=0 velocity=0.1
- joint arm_center_j0: origin xyz=-0.05908 0 0.44528 rpy=0 0 0 -> xyz=0 0.03852 0.25982 rpy=0 0 -1.57079; parent torso_l3 -> torso_flip_link

File: robots/humanoid/vega_1u/vega_1u_f5d6_collision_spheres.collision.urdf (robot description, URDF)
Before this commit: robot vega_1u_f5d6, 60 links, 59 joints
Links:
- removed link torso_l3
- added link base_link, mass 18.91029; visual mesh filename=meshes/visual/base_link.glb
- added link lift_link, mass 4.35777; collision sphere radius=0.09000000357627869; collision sphere radius=0.10999999940395355
- added link torso_flip_link, mass 0.71794; collision sphere radius=0.07999999821186066; collision sphere radius=0.07999999821186066
Joints:
- added joint Lift: type prismatic, parent base_link, child lift_link, origin xyz=0 0 0.01 rpy=0 0 0, axis 0 0 1, limit lower=0 upper=0.4 effort=0 velocity=0.05
- added joint torso_flip: type revolute, parent lift_link, child torso_flip_link, origin xyz=0 -0.06187 0.786 rpy=0 0 0, axis 1 0 0, limit lower=0 upper=1 effort=0 velocity=0.1
- joint arm_center_j0: origin xyz=-0.05908 0 0.44528 rpy=0 0 0 -> xyz=0 0.03852 0.25982 rpy=0 0 -1.57079; parent torso_l3 -> torso_flip_link

File: robots/humanoid/vega_1u/vega_1u_gripper.urdf (robot description, URDF)
Before this commit: robot vega_1u_gripper, 32 links, 31 joints
Links:
- removed link torso_l3
- added link base_link, mass 18.91029; collision mesh filename=meshes/visual/base_link.glb; visual mesh filename=meshes/visual/base_link.glb
- added link lift_link, mass 4.35777; collision mesh filename=meshes/visual/lift_link.glb; visual mesh filename=meshes/visual/lift_link.glb
- added link torso_flip_link, mass 0.71794; collision mesh filename=meshes/visual/torso_link.glb; visual mesh filename=meshes/visual/torso_link.glb
Joints:
- added joint Lift: type prismatic, parent base_link, child lift_link, origin xyz=0 0 0.01 rpy=0 0 0, axis 0 0 1, limit lower=0 upper=0.4 effort=0 velocity=0.05
- added joint torso_flip: type revolute, parent lift_link, child torso_flip_link, origin xyz=0 -0.06187 0.786 rpy=0 0 0, axis 1 0 0, limit lower=0 upper=1 effort=0 velocity=0.1
- joint arm_center_j0: origin xyz=-0.05908 0 0.44528 rpy=0 0 0 -> xyz=0 0.03852 0.25982 rpy=0 0 -1.57079; parent torso_l3 -> torso_flip_link

File: robots/humanoid/vega_1u/vega_1u_gripper_collision_spheres.collision.urdf (robot description, URDF)
Before this commit: robot vega_1u_gripper, 32 links, 31 joints
Links:
- removed link torso_l3
- added link base_link, mass 18.91029; visual mesh filename=meshes/visual/base_link.glb
- added link lift_link, mass 4.35777; collision sphere radius=0.09000000357627869; collision sphere radius=0.10999999940395355
- added link torso_flip_link, mass 0.71794; collision sphere radius=0.07999999821186066; collision sphere radius=0.07999999821186066
Joints:
- added joint Lift: type prismatic, parent base_link, child lift_link, origin xyz=0 0 0.01 rpy=0 0 0, axis 0 0 1, limit lower=0 upper=0.4 effort=0 velocity=0.05
- added joint torso_flip: type revolute, parent lift_link, child torso_flip_link, origin xyz=0 -0.06187 0.786 rpy=0 0 0, axis 1 0 0, limit lower=0 upper=1 effort=0 velocity=0.1
- joint arm_center_j0: origin xyz=-0.05908 0 0.44528 rpy=0 0 0 -> xyz=0 0.03852 0.25982 rpy=0 0 -1.57079; parent torso_l3 -> torso_flip_link
