Commit message: [release] (bot) Prepare public release 0.8.4
- Source commit: 3a4ffc2b35645bd2d5d2b5475b7af824a93832ab
- Generated: 2026-07-02 17:23:24 UTC
- Triggered by tag: refs/tags/v0.8.4

File: robots/humanoid/vega_1/vega_1_gripper.urdf (robot description, URDF)
Before this commit: robot vega_1_gripper, 51 links, 50 joints
Links:
- added link L_camera_link, mass 0.0253335276780861; visual mesh filename=../../hands/dexs_gripper/meshes/visual/camera_link.glb
- added link R_camera_link, mass 0.0253335276780861; visual mesh filename=../../hands/dexs_gripper/meshes/visual/camera_link.glb
- link L_gripper_base: mass 0.39258 -> 0.217869646528476; geometry collision mesh filename=../../hands/dexs_gripper/meshes/collision/gripper_base.obj; visual mesh filename=../../hands/dexs_gripper/meshes/visual/gripper_base.glb
- link L_gripper_l1: mass 0.09974 -> 0.0417789910080777; geometry collision mesh filename=../../hands/dexs_gripper/meshes/collision/gripper_l1.obj; visual mesh filename=../../hands/dexs_gripper/meshes/visual/gripper_l1.glb
- link L_gripper_l2: mass 0.09973 -> 0.0417790873345589; geometry collision mesh filename=../../hands/dexs_gripper/meshes/collision/gripper_l2.obj; visual mesh filename=../../hands/dexs_gripper/meshes/visual/gripper_l2.glb
- link R_gripper_base: mass 0.39258 -> 0.217869646528476; geometry collision mesh filename=../../hands/dexs_gripper/meshes/collision/gripper_base.obj; visual mesh filename=../../hands/dexs_gripper/meshes/visual/gripper_base.glb
- link R_gripper_l1: mass 0.09974 -> 0.0417789910080777; geometry collision mesh filename=../../hands/dexs_gripper/meshes/collision/gripper_l1.obj; visual mesh filename=../../hands/dexs_gripper/meshes/visual/gripper_l1.glb
- link R_gripper_l2: mass 0.09973 -> 0.0417790873345589; geometry collision mesh filename=../../hands/dexs_gripper/meshes/collision/gripper_l2.obj; visual mesh filename=../../hands/dexs_gripper/meshes/visual/gripper_l2.glb
Joints:
- added joint L_camera_joint: type fixed, parent L_gripper_base, child L_camera_link, origin xyz=0.0002 -0.07459 0.0017504 rpy=-0.087266 0 0
- added joint R_camera_joint: type fixed, parent R_gripper_base, child R_camera_link, origin xyz=0.0002 -0.07459 0.0017504 rpy=-0.087266 0 0
- joint L_gripper_j1: axis -1 0 0 -> 0 -1 0; origin xyz=4.92002E-18 0.0258 0.02875 rpy=0 0 0 -> xyz=-0.025807 -0.0015 0.02935 rpy=0 0 0
- joint L_gripper_j2: axis 1 0 0 -> 0 1 0; origin xyz=-1.39916E-18 -0.0258 0.02875 rpy=0 0 0 -> xyz=0.025793 -0.0015 0.02935 rpy=0 0 0
- joint L_hand_mount: origin xyz=0.0 0 0.078 rpy=0 0 0 -> xyz=0.0 0 0.0825 rpy=0 0 -1.5708
- joint R_gripper_j1: axis -1 0 0 -> 0 -1 0; origin xyz=4.92002E-18 0.0258 0.02875 rpy=0 0 0 -> xyz=-0.025807 -0.0015 0.02935 rpy=0 0 0
- joint R_gripper_j2: axis 1 0 0 -> 0 1 0; origin xyz=-1.39916E-18 -0.0258 0.02875 rpy=0 0 0 -> xyz=0.025793 -0.0015 0.02935 rpy=0 0 0
- joint R_hand_mount: origin xyz=0 0 0.078 rpy=0 0 0 -> xyz=0 0 0.0825 rpy=0 0 -1.5708

File: robots/humanoid/vega_1/vega_1_gripper_collision_spheres.collision.urdf (robot description, URDF)
Before this commit: robot vega_1_gripper, 51 links, 50 joints
Links:
- added link L_camera_link, mass 0.0253335276780861; visual mesh filename=../../hands/dexs_gripper/meshes/visual/camera_link.glb
- added link R_camera_link, mass 0.0253335276780861; visual mesh filename=../../hands/dexs_gripper/meshes/visual/camera_link.glb
- link L_gripper_base: mass 0.39258 -> 0.217869646528476; geometry collision sphere radius=0.029999999329447746; collision sphere radius=0.03999999910593033
- link L_gripper_l1: mass 0.09974 -> 0.0417789910080777; geometry collision sphere radius=0.01700000010430813; collision sphere radius=0.019999999664723874
- link L_gripper_l2: mass 0.09973 -> 0.0417790873345589; geometry collision sphere radius=0.01700000010430813; collision sphere radius=0.019999999664723874
- link R_gripper_base: mass 0.39258 -> 0.217869646528476; geometry collision sphere radius=0.029999999329447746; collision sphere radius=0.03999999910593033
- link R_gripper_l1: mass 0.09974 -> 0.0417789910080777; geometry collision sphere radius=0.01700000010430813; collision sphere radius=0.019999999664723874
- link R_gripper_l2: mass 0.09973 -> 0.0417790873345589; geometry collision sphere radius=0.01700000010430813; collision sphere radius=0.019999999664723874
Joints:
- added joint L_camera_joint: type fixed, parent L_gripper_base, child L_camera_link, origin xyz=0.0002 -0.07459 0.0017504 rpy=-0.087266 0 0
- added joint R_camera_joint: type fixed, parent R_gripper_base, child R_camera_link, origin xyz=0.0002 -0.07459 0.0017504 rpy=-0.087266 0 0
- joint L_gripper_j1: axis -1 0 0 -> 0 -1 0; origin xyz=4.92002E-18 0.0258 0.02875 rpy=0 0 0 -> xyz=-0.025807 -0.0015 0.02935 rpy=0 0 0
- joint L_gripper_j2: axis 1 0 0 -> 0 1 0; origin xyz=-1.39916E-18 -0.0258 0.02875 rpy=0 0 0 -> xyz=0.025793 -0.0015 0.02935 rpy=0 0 0
- joint L_hand_mount: origin xyz=0.0 0 0.078 rpy=0 0 0 -> xyz=0.0 0 0.0825 rpy=0 0 -1.5708
- joint R_gripper_j1: axis -1 0 0 -> 0 -1 0; origin xyz=4.92002E-18 0.0258 0.02875 rpy=0 0 0 -> xyz=-0.025807 -0.0015 0.02935 rpy=0 0 0
- joint R_gripper_j2: axis 1 0 0 -> 0 1 0; origin xyz=-1.39916E-18 -0.0258 0.02875 rpy=0 0 0 -> xyz=0.025793 -0.0015 0.02935 rpy=0 0 0
- joint R_hand_mount: origin xyz=0 0 0.078 rpy=0 0 0 -> xyz=0 0 0.0825 rpy=0 0 -1.5708

File: robots/humanoid/vega_1p/vega_1p_gripper.urdf (robot description, URDF)
Before this commit: robot vega_1p_gripper, 47 links, 46 joints
Links:
- added link L_camera_link, mass 0.0253335276780861; visual mesh filename=../../hands/dexs_gripper/meshes/visual/camera_link.glb
- added link R_camera_link, mass 0.0253335276780861; visual mesh filename=../../hands/dexs_gripper/meshes/visual/camera_link.glb
- link L_gripper_base: mass 0.39258 -> 0.217869646528476; geometry collision mesh filename=../../hands/dexs_gripper/meshes/collision/gripper_base.obj; visual mesh filename=../../hands/dexs_gripper/meshes/visual/gripper_base.glb
- link L_gripper_l1: mass 0.09974 -> 0.0417789910080777; geometry collision mesh filename=../../hands/dexs_gripper/meshes/collision/gripper_l1.obj; visual mesh filename=../../hands/dexs_gripper/meshes/visual/gripper_l1.glb
- link L_gripper_l2: mass 0.09973 -> 0.0417790873345589; geometry collision mesh filename=../../hands/dexs_gripper/meshes/collision/gripper_l2.obj; visual mesh filename=../../hands/dexs_gripper/meshes/visual/gripper_l2.glb
- link R_gripper_base: mass 0.39258 -> 0.217869646528476; geometry collision mesh filename=../../hands/dexs_gripper/meshes/collision/gripper_base.obj; visual mesh filename=../../hands/dexs_gripper/meshes/visual/gripper_base.glb
- link R_gripper_l1: mass 0.09974 -> 0.0417789910080777; geometry collision mesh filename=../../hands/dexs_gripper/meshes/collision/gripper_l1.obj; visual mesh filename=../../hands/dexs_gripper/meshes/visual/gripper_l1.glb
- link R_gripper_l2: mass 0.09973 -> 0.0417790873345589; geometry collision mesh filename=../../hands/dexs_gripper/meshes/collision/gripper_l2.obj; visual mesh filename=../../hands/dexs_gripper/meshes/visual/gripper_l2.glb
Joints:
- added joint L_camera_joint: type fixed, parent L_gripper_base, child L_camera_link, origin xyz=0.0002 -0.07459 0.0017504 rpy=-0.087266 0 0
- added joint R_camera_joint: type fixed, parent R_gripper_base, child R_camera_link, origin xyz=0.0002 -0.07459 0.0017504 rpy=-0.087266 0 0
- joint L_gripper_j1: axis -1 0 0 -> 0 -1 0; origin xyz=4.92002E-18 0.0258 0.02875 rpy=0 0 0 -> xyz=-0.025807 -0.0015 0.02935 rpy=0 0 0
- joint L_gripper_j2: axis 1 0 0 -> 0 1 0; origin xyz=-1.39916E-18 -0.0258 0.02875 rpy=0 0 0 -> xyz=0.025793 -0.0015 0.02935 rpy=0 0 0
- joint L_hand_mount: origin xyz=0.0 0 0.078 rpy=0 0 0 -> xyz=0.0 0 0.0825 rpy=0 0 -1.5708
- joint R_gripper_j1: axis -1 0 0 -> 0 -1 0; origin xyz=4.92002E-18 0.0258 0.02875 rpy=0 0 0 -> xyz=-0.025807 -0.0015 0.02935 rpy=0 0 0
- joint R_gripper_j2: axis 1 0 0 -> 0 1 0; origin xyz=-1.39916E-18 -0.0258 0.02875 rpy=0 0 0 -> xyz=0.025793 -0.0015 0.02935 rpy=0 0 0
- joint R_hand_mount: origin xyz=0 0 0.078 rpy=0 0 0 -> xyz=0 0 0.0825 rpy=0 0 -1.5708

File: robots/humanoid/vega_1p/vega_1p_gripper_collision_spheres.collision.urdf (robot description, URDF)
Before this commit: robot vega_1p_gripper, 47 links, 46 joints
Links:
- added link L_camera_link, mass 0.0253335276780861; visual mesh filename=../../hands/dexs_gripper/meshes/visual/camera_link.glb
- added link R_camera_link, mass 0.0253335276780861; visual mesh filename=../../hands/dexs_gripper/meshes/visual/camera_link.glb
- link L_gripper_base: mass 0.39258 -> 0.217869646528476; geometry collision sphere radius=0.029999999329447746; collision sphere radius=0.03999999910593033
- link L_gripper_l1: mass 0.09974 -> 0.0417789910080777; geometry collision sphere radius=0.01700000010430813; collision sphere radius=0.019999999664723874
- link L_gripper_l2: mass 0.09973 -> 0.0417790873345589; geometry collision sphere radius=0.01700000010430813; collision sphere radius=0.019999999664723874
- link R_gripper_base: mass 0.39258 -> 0.217869646528476; geometry collision sphere radius=0.029999999329447746; collision sphere radius=0.03999999910593033
- link R_gripper_l1: mass 0.09974 -> 0.0417789910080777; geometry collision sphere radius=0.01700000010430813; collision sphere radius=0.019999999664723874
- link R_gripper_l2: mass 0.09973 -> 0.0417790873345589; geometry collision sphere radius=0.01700000010430813; collision sphere radius=0.019999999664723874
Joints:
- added joint L_camera_joint: type fixed, parent L_gripper_base, child L_camera_link, origin xyz=0.0002 -0.07459 0.0017504 rpy=-0.087266 0 0
- added joint R_camera_joint: type fixed, parent R_gripper_base, child R_camera_link, origin xyz=0.0002 -0.07459 0.0017504 rpy=-0.087266 0 0
- joint L_gripper_j1: axis -1 0 0 -> 0 -1 0; origin xyz=4.92002E-18 0.0258 0.02875 rpy=0 0 0 -> xyz=-0.025807 -0.0015 0.02935 rpy=0 0 0
- joint L_gripper_j2: axis 1 0 0 -> 0 1 0; origin xyz=-1.39916E-18 -0.0258 0.02875 rpy=0 0 0 -> xyz=0.025793 -0.0015 0.02935 rpy=0 0 0
- joint L_hand_mount: origin xyz=0.0 0 0.078 rpy=0 0 0 -> xyz=0.0 0 0.0825 rpy=0 0 -1.5708
- joint R_gripper_j1: axis -1 0 0 -> 0 -1 0; origin xyz=4.92002E-18 0.0258 0.02875 rpy=0 0 0 -> xyz=-0.025807 -0.0015 0.02935 rpy=0 0 0
- joint R_gripper_j2: axis 1 0 0 -> 0 1 0; origin xyz=-1.39916E-18 -0.0258 0.02875 rpy=0 0 0 -> xyz=0.025793 -0.0015 0.02935 rpy=0 0 0
- joint R_hand_mount: origin xyz=0 0 0.078 rpy=0 0 0 -> xyz=0 0 0.0825 rpy=0 0 -1.5708

File: robots/humanoid/vega_1u/vega_1u_gripper.urdf (robot description, URDF)
Before this commit: robot vega_1u_gripper, 34 links, 33 joints
Links:
- added link L_camera_link, mass 0.0253335276780861; visual mesh filename=../../hands/dexs_gripper/meshes/visual/camera_link.glb
- added link R_camera_link, mass 0.0253335276780861; visual mesh filename=../../hands/dexs_gripper/meshes/visual/camera_link.glb
- link L_gripper_base: mass 0.39258 -> 0.217869646528476; geometry collision mesh filename=../../hands/dexs_gripper/meshes/collision/gripper_base.obj; visual mesh filename=../../hands/dexs_gripper/meshes/visual/gripper_base.glb
- link L_gripper_l1: mass 0.09974 -> 0.0417789910080777; geometry collision mesh filename=../../hands/dexs_gripper/meshes/collision/gripper_l1.obj; visual mesh filename=../../hands/dexs_gripper/meshes/visual/gripper_l1.glb
- link L_gripper_l2: mass 0.09973 -> 0.0417790873345589; geometry collision mesh filename=../../hands/dexs_gripper/meshes/collision/gripper_l2.obj; visual mesh filename=../../hands/dexs_gripper/meshes/visual/gripper_l2.glb
- link R_gripper_base: mass 0.39258 -> 0.217869646528476; geometry collision mesh filename=../../hands/dexs_gripper/meshes/collision/gripper_base.obj; visual mesh filename=../../hands/dexs_gripper/meshes/visual/gripper_base.glb
- link R_gripper_l1: mass 0.09974 -> 0.0417789910080777; geometry collision mesh filename=../../hands/dexs_gripper/meshes/collision/gripper_l1.obj; visual mesh filename=../../hands/dexs_gripper/meshes/visual/gripper_l1.glb
- link R_gripper_l2: mass 0.09973 -> 0.0417790873345589; geometry collision mesh filename=../../hands/dexs_gripper/meshes/collision/gripper_l2.obj; visual mesh filename=../../hands/dexs_gripper/meshes/visual/gripper_l2.glb
Joints:
- added joint L_camera_joint: type fixed, parent L_gripper_base, child L_camera_link, origin xyz=0.0002 -0.07459 0.0017504 rpy=-0.087266 0 0
- added joint R_camera_joint: type fixed, parent R_gripper_base, child R_camera_link, origin xyz=0.0002 -0.07459 0.0017504 rpy=-0.087266 0 0
- joint L_gripper_j1: axis -1 0 0 -> 0 -1 0; origin xyz=4.92002E-18 0.0258 0.02875 rpy=0 0 0 -> xyz=-0.025807 -0.0015 0.02935 rpy=0 0 0
- joint L_gripper_j2: axis 1 0 0 -> 0 1 0; origin xyz=-1.39916E-18 -0.0258 0.02875 rpy=0 0 0 -> xyz=0.025793 -0.0015 0.02935 rpy=0 0 0
- joint L_hand_mount: origin xyz=0.0 0 0.078 rpy=0 0 0 -> xyz=0.0 0 0.0825 rpy=0 0 -1.5708
- joint R_gripper_j1: axis -1 0 0 -> 0 -1 0; origin xyz=4.92002E-18 0.0258 0.02875 rpy=0 0 0 -> xyz=-0.025807 -0.0015 0.02935 rpy=0 0 0
- joint R_gripper_j2: axis 1 0 0 -> 0 1 0; origin xyz=-1.39916E-18 -0.0258 0.02875 rpy=0 0 0 -> xyz=0.025793 -0.0015 0.02935 rpy=0 0 0
- joint R_hand_mount: origin xyz=0 0 0.078 rpy=0 0 0 -> xyz=0 0 0.0825 rpy=0 0 -1.5708

File: robots/humanoid/vega_1u/vega_1u_gripper_collision_spheres.collision.urdf (robot description, URDF)
Before this commit: robot vega_1u_gripper, 34 links, 33 joints
Links:
- added link L_camera_link, mass 0.0253335276780861; visual mesh filename=../../hands/dexs_gripper/meshes/visual/camera_link.glb
- added link R_camera_link, mass 0.0253335276780861; visual mesh filename=../../hands/dexs_gripper/meshes/visual/camera_link.glb
- link L_gripper_base: mass 0.39258 -> 0.217869646528476; geometry collision sphere radius=0.029999999329447746; collision sphere radius=0.03999999910593033
- link L_gripper_l1: mass 0.09974 -> 0.0417789910080777; geometry collision sphere radius=0.01700000010430813; collision sphere radius=0.019999999664723874
- link L_gripper_l2: mass 0.09973 -> 0.0417790873345589; geometry collision sphere radius=0.01700000010430813; collision sphere radius=0.019999999664723874
- link R_gripper_base: mass 0.39258 -> 0.217869646528476; geometry collision sphere radius=0.029999999329447746; collision sphere radius=0.03999999910593033
- link R_gripper_l1: mass 0.09974 -> 0.0417789910080777; geometry collision sphere radius=0.01700000010430813; collision sphere radius=0.019999999664723874
- link R_gripper_l2: mass 0.09973 -> 0.0417790873345589; geometry collision sphere radius=0.01700000010430813; collision sphere radius=0.019999999664723874
Joints:
- added joint L_camera_joint: type fixed, parent L_gripper_base, child L_camera_link, origin xyz=0.0002 -0.07459 0.0017504 rpy=-0.087266 0 0
- added joint R_camera_joint: type fixed, parent R_gripper_base, child R_camera_link, origin xyz=0.0002 -0.07459 0.0017504 rpy=-0.087266 0 0
- joint L_gripper_j1: axis -1 0 0 -> 0 -1 0; origin xyz=4.92002E-18 0.0258 0.02875 rpy=0 0 0 -> xyz=-0.025807 -0.0015 0.02935 rpy=0 0 0
- joint L_gripper_j2: axis 1 0 0 -> 0 1 0; origin xyz=-1.39916E-18 -0.0258 0.02875 rpy=0 0 0 -> xyz=0.025793 -0.0015 0.02935 rpy=0 0 0
- joint L_hand_mount: origin xyz=0.0 0 0.078 rpy=0 0 0 -> xyz=0.0 0 0.0825 rpy=0 0 -1.5708
- joint R_gripper_j1: axis -1 0 0 -> 0 -1 0; origin xyz=4.92002E-18 0.0258 0.02875 rpy=0 0 0 -> xyz=-0.025807 -0.0015 0.02935 rpy=0 0 0
- joint R_gripper_j2: axis 1 0 0 -> 0 1 0; origin xyz=-1.39916E-18 -0.0258 0.02875 rpy=0 0 0 -> xyz=0.025793 -0.0015 0.02935 rpy=0 0 0
- joint R_hand_mount: origin xyz=0 0 0.078 rpy=0 0 0 -> xyz=0 0 0.0825 rpy=0 0 -1.5708
